File: co2monitor.kicad_pcb (KiCad board)
At the start: 2 copper layers, 70 x 70 mm, 40 parts, among them J1 USB_C_Receptacle_USB2.0, J2 UART, J3 I2C, J4 5V, J5 JTAG, SW1 RESET, SW2 BOOT, U1 AP2112K-3.3, U2 ESP32-S3-WROOM-1, U3 BME680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

Commit message: Don't silkscreen "Antenna Area" outside board
Routing:
- net GND: vias 36 -> 42
Changed lines of the file:
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@@
     )
     (fp_line (start -9 9) (end -9 9.75) (layer "F.SilkS") (width 0.12))
-    (fp_line (start -9 -15.75) (end 9 -15.75) (layer "F.SilkS") (width 0.12))
     (fp_line (start 9 9.75) (end 8 9.75) (layer "F.SilkS") (width 0.12))
-    (fp_line (start -9 -15.75) (end -9 -9) (layer "F.SilkS") (width 0.12))
     (fp_line (start -9 9.75) (end -8 9.75) (layer "F.SilkS") (width 0.12))
-    (fp_line (start 9 -15.75) (end 9 -9) (layer "F.SilkS") (width 0.12))
-    (fp_line (start 9 -9.81) (end -9 -9.81) (layer "F.SilkS") (width 0.12))
     (fp_line (start 9 9) (end 9 9.75) (layer "F.SilkS") (width 0.12))
     (fp_line (start 9 9.75) (end -9 9.75) (layer "Eco2.User") (width 0.12))
-    (fp_line (start 9 -15.75) (end 9 9.75) (layer "Eco2.User") (width 0.12))
+    (fp_line (start 9 -9.81) (end 9 9.75) (layer "Eco2.User") (width 0.12))
     (fp_line (start -9 -9.81) (end 9 -9.81) (layer "Eco2.User") (width 0.12))
-    (fp_line (start -9 9.75) (end -9 -15.75) (layer "Eco2.User") (width 0.12))
-    (fp_line (start -9 -15.75) (end 9 -15.75) (layer "Eco2.User") (width 0.12))
+    (fp_line (start -9 9.75) (end -9 -9.81) (layer "Eco2.User") (width 0.12))
     (fp_line (start -9.8 10.55) (end 9.8 10.55) (layer "F.CrtYd") (width 0.12))
     (fp_line (start 9.8 -16.05) (end 9.8 10.55) (layer "F.CrtYd") (width 0.12))
     (fp_line (start 9.8 -16.05) (end -9.8 -16.05) (layer "F.CrtYd") (width 0.12))
     (fp_line (start -9.8 -16.05) (end -9.8 10.55) (layer "F.CrtYd") (width 0.12))
+    (fp_line (start -9 -15.75) (end 9 -15.75) (layer "F.Fab") (width 0.12))
+    (fp_line (start -9 -15.75) (end -9 -9.81) (layer "F.Fab") (width 0.12))
+    (fp_line (start 9 -15.75) (end 9 -9.81) (layer "F.Fab") (width 0.12))
+    (fp_line (start 9 -9.81) (end -9 -9.81) (layer "F.Fab") (width 0.12))
     (pad "1" smd rect locked (at -8.75 -8.26) (size 1.5 0.9) (layers "F.Cu" "F.Paste" "F.Mask")
       (net 1 "GND") (pinfunction "GND") (pintype "power_in"))
@@
   (via (at 129.4 104.1) (size 0.8) (drill 0.4) (layers "F.Cu" "B.Cu") (free) (net 1))
   (via (at 108.3 110.8) (size 0.8) (drill 0.4) (layers "F.Cu" "B.Cu") (free) (net 1))
+  (via (at 162.3 75) (size 0.8) (drill 0.4) (layers "F.Cu" "B.Cu") (free) (net 1))
   (via (at 149.8 107.4) (size 0.8) (drill 0.4) (layers "F.Cu" "B.Cu") (free) (net 1))
   (via (at 140.4 125.8) (size 0.8) (drill 0.4) (layers "F.Cu" "B.Cu") (free) (net 1))
@@
   (via (at 142.4 93.4) (size 0.8) (drill 0.4) (layers "F.Cu" "B.Cu") (free) (net 1))
   (via (at 132.1 92) (size 0.8) (drill 0.4) (layers "F.Cu" "B.Cu") (free) (net 1))
+  (via (at 159.8 79.2) (size 0.8) (drill 0.4) (layers "F.Cu" "B.Cu") (free) (net 1))
   (via (at 113.4 136.8) (size 0.8) (drill 0.4) (layers "F.Cu" "B.Cu") (free) (net 1))
   (via (at 148 82.1) (size 0.8) (drill 0.4) (layers "F.Cu" "B.Cu") (free) (net 1))
   (via (at 108.4 81.6) (size 0.8) (drill 0.4) (layers "F.Cu" "B.Cu") (free) (net 1))
   (via (at 130.3 112.2) (size 0.8) (drill 0.4) (layers "F.Cu" "B.Cu") (free) (net 1))
+  (via (at 158.5 99.1) (size 0.8) (drill 0.4) (layers "F.Cu" "B.Cu") (free) (net 1))
   (via (at 121 104.1) (size 0.8) (drill 0.4) (layers "F.Cu" "B.Cu") (free) (net 1))
   (via (at 158.5 129) (size 0.8) (drill 0.4) (layers "F.Cu" "B.Cu") (free) (net 1))
@@
   (via (at 114.3 115.4) (size 0.8) (drill 0.4) (layers "F.Cu" "B.Cu") (free) (net 1))
   (via (at 126.9 130.5) (size 0.8) (drill 0.4) (layers "F.Cu" "B.Cu") (free) (net 1))
+  (via (at 154.6 85.9) (size 0.8) (drill 0.4) (layers "F.Cu" "B.Cu") (free) (net 1))
+  (via (at 167.7 78.3) (size 0.8) (drill 0.4) (layers "F.Cu" "B.Cu") (free) (net 1))
   (via (at 135.3 96.1) (size 0.8) (drill 0.4) (layers "F.Cu" "B.Cu") (free) (net 1))
   (via (at 131.4 107.5) (size 0.8) (drill 0.4) (layers "F.Cu" "B.Cu") (free) (net 1))
@@
   (via (at 140.7 120.1) (size 0.8) (drill 0.4) (layers "F.Cu" "B.Cu") (free) (net 1))
   (via (at 107.7 124.8) (size 0.8) (drill 0.4) (layers "F.Cu" "B.Cu") (free) (net 1))
+  (via (at 168.7 89.8) (size 0.8) (drill 0.4) (layers "F.Cu" "B.Cu") (free) (net 1))
   (via (at 126.5 87.7) (size 0.8) (drill 0.4) (layers "F.Cu" "B.Cu") (free) (net 1))
   (via (at 131 100.8) (size 0.8) (drill 0.4) (layers "F.Cu" "B.Cu") (free) (net 1))
